File: PCB/speek_rx/speek_rx.kicad_sch (KiCad schematic)
At the start: 69 parts, among them CN1 PJ-320D, CN2 PJ-320D, J1 Conn_01x02, J3 Conn_01x06_Socket, J4 Conn_01x04, SW1 TS-1187A-B-A-B, SW2 TS-1187A-B-A-B, U1 ESP32-D0WD-V3, U2 W25Q32JVSSIQ_C179173, U3 CP2102N-A02-GQFN24R, U4 SPX1117M3-L-3-3/TR, U5 PCM5102APW, U6 TPA6132A2RTER, X1 XL2EL89CPI-111YLC-40M

Commit message: routing
Parts:
- renumbered SW1 to BOOT1, SW2 to EN1
Changed lines of the file:
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@@
 		(dnp no)
 		(fields_autoplaced yes)
-		(property "Reference" "SW2"
+		(property "Reference" "EN1"
 			(at 76.2 137.16 0)
 			(show_name no)
@@
 			(project "speek_rx"
 				(path "/75a8527f-6d13-4893-9d8d-0dff56ab3f3e"
-					(reference "SW2")
+					(reference "EN1")
 					(unit 1)
 				)
@@
 		(dnp no)
 		(fields_autoplaced yes)
-		(property "Reference" "SW1"
+		(property "Reference" "BOOT1"
 			(at 48.26 137.16 0)
 			(show_name no)
@@
 			(project "speek_rx"
 				(path "/75a8527f-6d13-4893-9d8d-0dff56ab3f3e"
-					(reference "SW1")
+					(reference "BOOT1")
 					(unit 1)
 				)

Commit message: bom-optimize
Parts:
- C21: LCSC Part C368809 -> C23733
- C6: LCSC Part C60133 -> C15195
- C7: LCSC Part C107028 -> C26404
- C9: LCSC Part C106200 -> C1546
- R1: LCSC Part C140184 -> C25765
- R3, R7: LCSC Part C60490 -> C25744
- R4: LCSC Part C106235 -> C11702
Changed lines of the file:
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@@
 			)
 		)
-		(property "LCSC Part" "C106235"
+		(property "LCSC Part" "C11702"
 			(at 168.91 184.15 0)
 			(hide yes)
@@
 			)
 		)
-		(property "LCSC Part" "C140184"
+		(property "LCSC Part" "C25765"
 			(at 142.24 71.12 0)
 			(hide yes)
@@
 			)
 		)
-		(property "LCSC Part" "C106200"
+		(property "LCSC Part" "C1546"
 			(at 163.83 81.28 0)
 			(hide yes)
@@
 			)
 		)
-		(property "LCSC Part" "C60490"
+		(property "LCSC Part" "C25744"
 			(at 38.1 128.27 0)
 			(hide yes)
@@
 			)
 		)
-		(property "LCSC Part" "C60490"
+		(property "LCSC Part" "C25744"
 			(at 125.73 187.96 0)
 			(hide yes)
@@
 			)
 		)
-		(property "LCSC Part" "C60133"
+		(property "LCSC Part" "C15195"
 			(at 132.08 82.55 0)
 			(hide yes)
@@
 			)
 		)
-		(property "LCSC Part" "C368809"
+		(property "LCSC Part" "C23733"
 			(at 142.24 173.99 0)
 			(hide yes)
@@
 			)
 		)
-		(property "LCSC Part" "C107028"
+		(property "LCSC Part" "C26404"
 			(at 99.06 69.85 0)
 			(hide yes)
