File: PCB/speek_rx/speek_rx.kicad_pcb (KiCad board)
At the start: 2 copper layers, 80 x 60 mm, 67 parts, among them CN1 PJ-320D, CN2 PJ-320D, J1 Conn_01x02, SW1 TS-1187A-B-A-B, SW2 TS-1187A-B-A-B, U1 ESP32-D0WD-V3, U2 W25Q32JVSSIQ_C179173, U3 CP2102N-A02-GQFN24R, U4 SPX1117M3-L-3-3/TR, U5 PCM5102APW, U6 TPA6132A2RTER, X1 XL2EL89CPI-111YLC-40M

Commit message: pcb placement done
Parts:
- moved C27 152.9 mm to (197.6, 73.5)
- moved C37 151.5 mm to (196.1, 78.5)
- moved C26 149.4 mm to (197.6, 72.5)
- moved C24 148.3 mm to (188.0, 70.6), turned to -90 degrees
- moved C28 146.7 mm to (188.6, 74.5)
- moved C29 146.6 mm to (188.6, 75.7)
- moved C8 142.5 mm to (175.6, 53.0)
- moved C12 140.7 mm to (177.5, 56.1), turned to 90 degrees
- moved C5 139.1 mm to (173.0, 61.9), turned to 90 degrees
- moved C25 138.8 mm to (189.0, 70.5), turned to -90 degrees
- moved C9 138.7 mm to (175.6, 54.0), turned to 180 degrees
- moved C2 135.6 mm to (169.5, 56.1), turned to 90 degrees
- moved C16 122.9 mm to (159.6, 62.0)
- moved C21 110.0 mm to (149.5, 55.4), turned to 90 degrees
- moved C20 108.7 mm to (148.3, 55.6), turned to 90 degrees
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
Commit message: start routing ig
Parts:
- added J3: Conn_01x06_Socket, Connector_PinHeader_2.54mm:PinHeader_1x06_P2.54mm_Horizontal, F.Cu at (172.2, 89.7)
- added J4: Conn_01x04, Connector_PinHeader_2.54mm:PinHeader_1x04_P2.54mm_Horizontal, F.Cu at (205.1, 46.2)
- moved C18 39.8 mm to (167.5, 86.6)
- moved C19 7.15 mm to (155.4, 86.6)
- moved SW1 7.15 mm to (162.9, 85.2)
- moved SW2 7.15 mm to (150.9, 85.0)
- moved C22 3.50 mm to (192.5, 63.1)
- moved C23 3.50 mm to (193.5, 63.1)
- moved C24 3.50 mm to (188.0, 67.1)
- moved C25 3.50 mm to (189.0, 67.0)
- moved C26 3.50 mm to (197.6, 69.0)
- moved C27 3.50 mm to (197.6, 70.0)
- moved C28 3.50 mm to (188.6, 71.0)
- moved C29 3.50 mm to (188.6, 72.2)
- moved C30 3.50 mm to (195.1, 73.5)
- moved C31 3.50 mm to (191.4, 73.5)
- moved C32 3.50 mm to (193.0, 74.4)
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Routing:
- net /VBUS: track 0.00 -> 43.9 mm
- net /CHIP_PU: track 0.00 -> 32.1 mm
- net /PVDD: track 0.00 -> 29.2 mm
- net /DTR: track 0.00 -> 17.7 mm
- net /D-: track 0.00 -> 6.61 mm
- net /D+: track 0.00 -> 6.59 mm
- net /__VBUS_U0P: track 0.00 -> 3.03 mm
- net Net-(U3-RSTb): track 0.00 -> 1.91 mm
- net /U0TXD: track 0.00 -> 1.50 mm

Commit message: lwk routed the whole thing
Parts:
- moved C13 1.64 mm to (175.9, 61.0)
- moved AE1 1.35 mm to (159.2, 37.5), turned to 90 degrees
- moved C8 0.50 mm to (175.6, 52.5)
- moved C9 0.50 mm to (175.6, 53.5)
- moved C6 0.25 mm to (172.4, 53.2)
- moved C35 0.17 mm to (194.5, 81.2)
- moved C11 0.08 mm to (174.0, 53.0)
Routing:
- net /PVDD: track 29.2 -> 176.0 mm, vias 0 -> 8
- net /U0RXD: track 0.00 -> 89.7 mm, vias 0 -> 2
- net /DTR: track 17.7 -> 102.7 mm, vias 0 -> 3
- net /CHIP_PU: track 32.1 -> 101.8 mm, vias 0 -> 1
- net /DIN: track 0.00 -> 55.3 mm, vias 0 -> 1
- net /U0TXD: track 1.50 -> 55.1 mm, vias 0 -> 1
- net GND: track 0.00 -> 53.5 mm, vias 0 -> 32
- net /GPIO25: track 0.00 -> 53.1 mm, vias 0 -> 2
- net /BCK: track 0.00 -> 48.3 mm, vias 0 -> 2
- net /OUTR: track 0.00 -> 41.0 mm, vias 0 -> 2
- net /VBUS: track 43.9 -> 76.5 mm, vias 0 -> 2
- net Net-(U1-U0TXD): track 0.00 -> 31.9 mm, vias 0 -> 2
- net /OUTL_FINAL: track 0.00 -> 31.4 mm
- net /OUTL: track 0.00 -> 25.2 mm, vias 0 -> 2
- net /AGND: track 0.00 -> 18.6 mm, vias 0 -> 2
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
Commit message: vanity vias lol
Routing:
- net GND: vias 32 -> 54
Changed lines of the file:
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@@
 		(capping no)
 		(filling no)
-		(zone_defaults)
 		(pcbplotparams
 			(layerselection 0x00000000_00000000_55555555_5755f5ff)
@@
 	)
 	(via
+		(at 183 49.5)
+		(size 0.6)
+		(drill 0.3)
+		(layers "F.Cu" "B.Cu")
+		(free yes)
+		(net "GND")
+	)
+	(via
 		(at 195.5 81.5)
 		(size 0.6)
@@
 	)
 	(via
+		(at 179 76)
+		(size 0.6)
+		(drill 0.3)
+		(layers "F.Cu" "B.Cu")
+		(free yes)
+		(net "GND")
+	)
+	(via
 		(at 170 61.25)
 		(size 0.6)
@@
 	)
 	(via
+		(at 184 57)
+		(size 0.6)
+		(drill 0.3)
+		(layers "F.Cu" "B.Cu")
+		(free yes)
+		(net "GND")
+	)
+	(via
 		(at 160.8 36.15)
 		(size 0.6)
@@
 	)
 	(via
+		(at 184.5 50.5)
+		(size 0.6)
+		(drill 0.3)
+		(layers "F.Cu" "B.Cu")
+		(free yes)
+		(net "GND")
+	)
+	(via
 		(at 169.5 57)
 		(size 0.6)
@@
 	)
 	(via
+		(at 183 59)
+		(size 0.6)
+		(drill 0.3)
+		(layers "F.Cu" "B.Cu")
+		(free yes)
+		(net "GND")
+	)
+	(via
 		(at 160.8 35.55)
 		(size 0.6)
@@
 	)
 	(via
+		(at 182.5 50)
+		(size 0.6)
+		(drill 0.3)
+		(layers "F.Cu" "B.Cu")
+		(free yes)
+		(net "GND")
+	)
+	(via
 		(at 160.8 33.8)
 		(size 0.6)
@@
 	)
 	(via
+		(at 182.5 58.5)
+		(size 0.6)
+		(drill 0.3)
+		(layers "F.Cu" "B.Cu")
+		(free yes)
+		(net "GND")
+	)
+	(via
+		(at 175 69.5)
+		(size 0.6)
+		(drill 0.3)
+		(layers "F.Cu" "B.Cu")
+		(free yes)
+		(net "GND")
+	)
+	(via
 		(at 160.8 34.95)
 		(size 0.6)
@@
 	)
 	(via
+		(at 180.5 75)
+		(size 0.6)
+		(drill 0.3)
+		(layers "F.Cu" "B.Cu")
+		(free yes)
+		(net "GND")
+	)
+	(via
 		(at 173.5 52.25)
 		(size 0.6)
@@
 	)
 	(via
+		(at 170 67)
+		(size 0.6)
+		(drill 0.3)
+		(layers "F.Cu" "B.Cu")
+		(free yes)
+		(net "GND")
+	)
+	(via
 		(at 177.3 50.25)
 		(size 0.6)
@@
 	)
 	(via
+		(at 182 58)
+		(size 0.6)
+		(drill 0.3)
+		(layers "F.Cu" "B.Cu")
+		(free yes)
+		(net "GND")
+	)
+	(via
+		(at 184 51)
+		(size 0.6)
+		(drill 0.3)
+		(layers "F.Cu" "B.Cu")
+		(free yes)
+		(net "GND")
+	)
+	(via
+		(at 173.5 71)
+		(size 0.6)
+		(drill 0.3)
+		(layers "F.Cu" "B.Cu")
+		(free yes)
+		(net "GND")
+	)
+	(via
 		(at 154.6 40.8)
 		(size 0.6)
@@
 	)
 	(via
+		(at 171 65.5)
+		(size 0.6)
+		(drill 0.3)
+		(layers "F.Cu" "B.Cu")
+		(free yes)
+		(net "GND")
+	)
+	(via
+		(at 183.5 56.5)
+		(size 0.6)
+		(drill 0.3)
+		(layers "F.Cu" "B.Cu")
+		(free yes)
+		(net "GND")
+	)
+	(via
+		(at 183.5 51.5)
+		(size 0.6)
+		(drill 0.3)
+		(layers "F.Cu" "B.Cu")
+		(free yes)
+		(net "GND")
+	)
+	(via
 		(at 193.5 78.25)
 		(size 0.6)
@@
 	)
 	(via
+		(at 178 75)
+		(size 0.6)
+		(drill 0.3)
+		(layers "F.Cu" "B.Cu")
+		(free yes)
+		(net "GND")
+	)
+	(via
+		(at 184.5 57.5)
+		(size 0.6)
+		(drill 0.3)
+		(layers "F.Cu" "B.Cu")
+		(free yes)
+		(net "GND")
+	)
+	(via
 		(at 160.8 34.35)
 		(size 0.6)
@@
 	)
 	(via
+		(at 180 74.5)
+		(size 0.6)
+		(drill 0.3)
+		(layers "F.Cu" "B.Cu")
+		(free yes)
+		(net "GND")
+	)
+	(via
 		(at 155.8 40.8)
 		(size 0.6)
@@
 	)
 	(via
+		(at 182 50.5)
+		(size 0.6)
+		(drill 0.3)
+		(layers "F.Cu" "B.Cu")
+		(free yes)
+		(net "GND")
+	)
+	(via
+		(at 179.5 74)
+		(size 0.6)
+		(drill 0.3)
+		(layers "F.Cu" "B.Cu")
+		(free yes)
+		(net "GND")
+	)
+	(via
 		(at 171.55 63.1)
 		(size 0.6)
@@
 		(net "GND")
 	)
+	(via
+		(at 178.5 75.5)
+		(size 0.6)
+		(drill 0.3)
+		(layers "F.Cu" "B.Cu")
+		(free yes)
+		(net "GND")
+	)

Commit message: routing
Parts:
- renumbered SW1 to BOOT, SW2 to EN
Routing:
- net GND: track 53.5 -> 56.4 mm, vias 54 -> 55
- net Net-(U6-INL-): track 4.72 -> 5.48 mm
- net /PVDD: track 176.0 -> 176.7 mm
Other:
- board text added: "*RX/TX flipped depending on how you think about it"
- board text added: "BCK"
- board text added: "DIN"
- board text added: "DTR"
- board text added: "EN"
- board text added: "GND"
- board text added: "GP25"
- board text added: "Headphones"
- board text added: "Line out"
- board text added: "RX*"
- board text added: "Speek RX"
- board text added: "TX*"
- board text added: "VBUS"

Commit message: Update speek_rx.kicad_pcb
Routing:
- net GND: track 56.4 -> 56.9 mm, vias 55 -> 56
Changed lines of the file:
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@@
 		)
 	)
-	(gr_text "GND"
-		(at 206.25 54.5 0)
+	(gr_text "GP25"
+		(at 201 46.75 0)
 		(layer "F.SilkS")
 		(effects
@@
 		)
 	)
-	(gr_text "GP25"
-		(at 206.5 46.75 0)
+	(gr_text "BCK"
+		(at 201.75 52 0)
 		(layer "F.SilkS")
 		(effects
@@
 		)
 	)
-	(gr_text "DIN"
-		(at 206.5 49.25 0)
+	(gr_text "GND"
+		(at 201.75 54.5 0)
 		(layer "F.SilkS")
 		(effects
@@
 		)
 	)
-	(gr_text "BCK"
-		(at 206.5 51.75 0)
+	(gr_text "DIN"
+		(at 204 49.25 0)
 		(layer "F.SilkS")
 		(effects
@@
 				(bold yes)
 			)
-			(justify left bottom)
+			(justify right bottom)
 		)
 	)
@@
 	)
 	(segment
+		(start 167.41 55.34)
+		(end 167.5 55.25)
+		(width 0.2)
+		(layer "F.Cu")
+		(net "GND")
+	)
+	(segment
 		(start 172.15 89.705)
 		(end 172.15 88.2)
@@
 	)
 	(segment
+		(start 167 55.34)
+		(end 167.41 55.34)
+		(width 0.2)
+		(layer "F.Cu")
+		(net "GND")
+	)
+	(segment
 		(start 176 53)
 		(end 176.50076 53)
@@
 	)
 	(segment
+		(start 167 55.34)
+		(end 167.04 55.34)
+		(width 0.2)
+		(layer "F.Cu")
+		(net "GND")
+	)
+	(segment
 		(start 193.25 76.75)
 		(end 193.25 78)
@@
 	(segment
 		(start 166.5 55.34)
-		(end 167.04 55.34)
+		(end 167 55.34)
 		(width 0.2)
 		(layer "F.Cu")
@@
 		(net "GND")
 	)
+	(via
+		(at 167.5 55.25)
+		(size 0.6)
+		(drill 0.3)
+		(layers "F.Cu" "B.Cu")
+		(net "GND")
+	)
