File: PCB/speek_split/speek_split.kicad_pcb (KiCad board)
At the start: 2 copper layers, 80 x 60 mm, 14 parts

Commit message: H
Parts:
- moved H2 52.0 mm to (214.3, 44.1)
- moved H3 52.0 mm to (142.3, 96.1)
- moved H4 52.0 mm to (214.3, 96.1)
- moved H1 51.9 mm to (142.3, 44.1)
