File: PCB/speek_split/speek_split.kicad_sch (KiCad schematic)
At the start: 10 parts

Commit message: H
Parts:
- added H1, H2, H3, H4: MountingHole, MountingHole:MountingHole_3.2mm_M3, symbol Mechanical:MountingHole
