File: speek-rx/PCB/speek_rx/speek_rx.kicad_pcb (KiCad board)
At the start: 2 copper layers, 80 x 60 mm, 69 parts, among them CN1 PJ-320D, CN2 PJ-320D, J1 Conn_01x02, J3 Conn_01x06_Socket, J4 Conn_01x04, U1 ESP32-D0WD-V3, U2 W25Q32JVSSIQ_C179173, U3 CP2102N-A02-GQFN24R, U4 SPX1117M3-L-3-3/TR, U5 PCM5102APW, U6 TPA6132A2RTER, X1 XL2EL89CPI-111YLC-40M

Commit message: JST and antenna
Parts:
- added C38: 1pF, easyeda2kicad:C0402, F.Cu at (162.3, 42.0)
- added D3: PMEG060V100EPDZ, easyeda2kicad:SOT1289_L5.8-W4.4-LS6.5-RD, F.Cu at (147.0, 76.1)
- added D4: PMEG060V100EPDZ, easyeda2kicad:SOT1289_L5.8-W4.4-LS6.5-RD, F.Cu at (146.6, 66.8)
- added JP1: U.FL-R-SMT-1, easyeda2kicad:RF-SMD_FRF05002-JSS103M, F.Cu at (165.5, 47.5)
- added L4: 3.9nH, easyeda2kicad:IND-SMD_L1.0-W0.5-2, F.Cu at (161.2, 40.8)
- added L5: 2.7nH, easyeda2kicad:L0402, F.Cu at (160.7, 43.0)
- added R9: RC0603JR-070RL, easyeda2kicad:R0603, F.Cu at (162.8, 44.2)
- J1: footprint Connector_JST:JST_EH_S2B-EH_1x02_P2.50mm_Horizontal -> Connector_JST:JST_VH_B2P-VH-B_1x02_P3.96mm_Vertical
- moved J1 5.96 mm to (140.2, 71.2), turned to -90 degrees
- moved C2 0.25 mm to (169.2, 56.1)
- renumbered BOOT to BOOT1, EN to EN1
Connections:
- C15 pad 2: Net-(AE1-ANT) -> Net-(JP1-SIG)
- J1 pad 2: /VBUS -> Net-(J1-Pin_2)
- J3 pad 2: /VBUS -> /__VIN
- L3 pad 1: Net-(AE1-ANT) -> Net-(JP1-SIG)
- U4 pad 3: /VBUS -> /__VIN
Routing:
- net /__VIN: track 0.00 -> 43.2 mm
- net /VBUS: track 76.5 -> 36.8 mm
- net Net-(AE1-ANT): track 17.0 -> 2.24 mm
- net Net-(JP1-SIG): track 0.00 -> 12.5 mm
- net Net-(J1-Pin_2): track 0.00 -> 6.98 mm
- net Net-(C38-Pad2): track 0.00 -> 2.27 mm
- net Net-(C38-Pad1): track 0.00 -> 1.22 mm
- net /U0RXD: track 89.7 -> 90.2 mm
- net GND: track 56.9 -> 57.0 mm, vias 56 -> 215
- net /U0TXD: vias 1 -> 2
- net /DIN: vias 1 -> 2

Commit message: RX I guess
Other:
- board text added: "prefer USBC!!!"
