File: speek-rx/PCB/speek_rx/speek_rx.kicad_pcb (KiCad board)
At the start: 2 copper layers, 80 x 60 mm, 76 parts, among them CN1 PJ-320D, CN2 PJ-320D, J1 Conn_01x02, J3 Conn_01x06_Socket, J4 Conn_01x04, U1 ESP32-D0WD-V3, U2 W25Q32JVSSIQ_C179173, U3 CP2102N-A02-GQFN24R, U4 SPX1117M3-L-3-3/TR, U5 PCM5102APW, U6 TPA6132A2RTER, X1 XL2EL89CPI-111YLC-40M

Commit message: speek RX new board!!
Parts:
- removed C1, C13, C8: 1uF, lcsc:C0402
- removed C10, C11: 15pf, lcsc:C0402
- removed C12, C17, C2, C3, C5: 0.1uF, lcsc:C0402
- removed C14: GRM1555C1H2R7BA01D, easyeda2kicad:C0402
- removed C15: GRM1555C1H2R0BA01D, easyeda2kicad:C0402
- removed C4: 10uF, lcsc:C0402
- removed C6: CC0402KRX7R9BB103, easyeda2kicad:C0402
- removed C7: CC0402KRX7R9BB332, easyeda2kicad:C0402
- removed C9: CC0402JRNPO9BN101, easyeda2kicad:C0402
- removed L1: LQG15HS2N0S02D, easyeda2kicad:L0402
- removed L2: 15nH, lcsc:L0402
- removed L3: LQG15HS2N7S02D, easyeda2kicad:L0402
- removed R1: RC-02K2002FT, easyeda2kicad:R0402
- removed R2: 499Ω, lcsc:R0402
- removed R3: RC0402FR-0710KL, easyeda2kicad:R0402
- removed U1: ESP32-D0WD-V3, easyeda2kicad:QFN-48_L5.0-W5.0-P0.35-BL-EP3.7
- removed U2: W25Q32JVSSIQ_C179173, easyeda2kicad:SOIC-8_L5.3-W5.3-P1.27-LS8.0-BL
- removed X1: XL2EL89CPI-111YLC-40M, lcsc:CRYSTAL-SMD_4P-L3.2-W2.5-BL
- added C39: 0.1uF, lcsc:C0402, F.Cu at (169.0, 55.5)
- added C40: 10uF, lcsc:C0402, F.Cu at (168.9, 56.8)
- added Q1: SS8050-G, easyeda2kicad:SOT-23-3_L2.9-W1.5-P1.90-LS2.6-BR, F.Cu at (166.4, 66.5)
- added Q2: SS8050-G, easyeda2kicad:SOT-23-3_L2.9-W1.5-P1.90-LS2.6-BR, F.Cu at (162.4, 66.5)
- added R10: 10k, easyeda2kicad:R0402, F.Cu at (163.1, 62.9)
- added R11: 10k, easyeda2kicad:R0402, F.Cu at (165.2, 68.8)
- added U19: ESP32-PICO-V3-02, easyeda2kicad:QFN-48_L7.0-W7.0-P0.50-BL-EP5.1, F.Cu at (174.2, 56.6)
Connections:
- BOOT1 pad 2: /DTR -> /GPIO0
- BOOT1 pad 4: /DTR -> /GPIO0
- C18 pad 1: /DTR -> /GPIO0
- J3 pad 4: /CHIP_PU -> /RTS
- JP1 pad 1: Net-(JP1-SIG) -> /LNA_IN
- R9 pad 2: Net-(JP1-SIG) -> /LNA_IN
- U3 pad 19: /CHIP_PU -> /RTS
Routing:
- net /CHIP_PU: track 101.8 -> 41.6 mm, vias 1 -> 2
- net /RTS: track 0.00 -> 57.0 mm, vias 0 -> 3
- net /GPIO0: track 0.00 -> 46.9 mm, vias 0 -> 4
- net /DTR: track 102.7 -> 62.8 mm, vias 3 -> 2
- net Net-(U1-U0TXD): track 32.1 -> 0.00 mm, vias 2 -> 0
- net /PVDD: track 176.7 -> 154.2 mm, vias 8 -> 2
- net GND: track 57.0 -> 37.7 mm, vias 215 -> 194
- net /U0TXD: track 55.1 -> 71.2 mm
- net Net-(JP1-SIG): track 12.5 -> 0.00 mm
- net /SCS: track 10.5 -> 0.00 mm, vias 2 -> 0
- net /VDD_SDIO: track 10.5 -> 0.00 mm
- net /LNA_IN: track 4.09 -> 14.4 mm
- net Net-(U1-CAP1): track 10.0 -> 0.00 mm
- net /U0RXD: track 90.2 -> 98.9 mm, vias 2 -> 3
- net /SD3: track 8.70 -> 0.00 mm, vias 2 -> 0
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
Commit message: aguihegwroiughawrg
Parts:
- removed D3, D4: PMEG060V100EPDZ, easyeda2kicad:SOT1289_L5.8-W4.4-LS6.5-RD
- removed J1: Conn_01x02, Connector_JST:JST_VH_B2P-VH-B_1x02_P3.96mm_Vertical
- C30, C31, C36, C37: value CL05A225KO5NQNC -> CL05A225MQ5NSNC
- D2: value PESD3V3L1BA,115 -> PESD3V3L1BA
- Q1, Q2: value SS8050-G -> SS8050
- R5: value AR02DTD4752 -> 47k
- R6: value CRCW040222K1FKED -> 22k
- R7: value RC0402FR-0710KL -> 10k
- R9: value RC0603JR-070RL -> 0R
- U4: value SPX1117M3-L-3-3/TR -> AMS1117-3.3
Connections:
- J3 pad 2: /__VIN -> /VBUS
- U4 pad 3: /__VIN -> /VBUS
Routing:
- net /__VIN: track 43.5 -> 0.00 mm
- net /VBUS: track 36.8 -> 76.2 mm
- net Net-(J1-Pin_2): track 6.68 -> 0.00 mm
Other:
- board text removed: "prefer USBC!!!"
