File: speek-rx/PCB/speek_rx/speek_rx.kicad_sch (KiCad schematic)
At the start: 69 parts, among them CN1 PJ-320D, CN2 PJ-320D, J1 Conn_01x02, J3 Conn_01x06_Socket, J4 Conn_01x04, U1 ESP32-D0WD-V3, U2 W25Q32JVSSIQ_C179173, U3 CP2102N-A02-GQFN24R, U4 SPX1117M3-L-3-3/TR, U5 PCM5102APW, U6 TPA6132A2RTER, X1 XL2EL89CPI-111YLC-40M

Commit message: JST and antenna
Parts:
- added C38: 1pF, easyeda2kicad:C0402, symbol lcsc:CC0402BRNPO9BN1R0
- added D3, D4: PMEG060V100EPDZ, easyeda2kicad:SOT1289_L5.8-W4.4-LS6.5-RD, symbol lcsc:PMEG060V100EPDZ
- added JP1: U.FL-R-SMT-1, easyeda2kicad:RF-SMD_FRF05002-JSS103M, symbol lcsc:U.FL-R-SMT-1
- added L4: 3.9nH, easyeda2kicad:IND-SMD_L1.0-W0.5-2, symbol lcsc:LQW15AN3N9B00D
- added L5: 2.7nH, easyeda2kicad:L0402, symbol lcsc:LQG15HS2N7S02D
- added R9: RC0603JR-070RL, easyeda2kicad:R0603, symbol lcsc:RC0603JR-070RL
- J1: footprint Connector_JST:JST_EH_S2B-EH_1x02_P2.50mm_Horizontal -> Connector_JST:JST_VH_B2P-VH-B_1x02_P3.96mm_Vertical
Connections:
- net GND: now also JP1.2 (GND), JP1.3 (GND), L5.1
- net VBUS: now also D4.1 (A), D4.2 (A); no longer J1.2 (Pin_2), J3.2 (Pin_2), U4.3 (input)
- net at C15.2, L3.1: now also JP1.1 (SIG), R9.2; no longer AE1.1 (ANT)
- new net: C38.1, R9.1
- new net: C38.2, L4.2, L5.2
- new net: D3.1 (A), D3.2 (A), J1.2 (Pin_2)
- new net: AE1.1 (ANT), L4.1
- new net __VIN: D3.3 (K), D4.3 (K), J3.2 (Pin_2), U4.3 (input)
Other:
- moved on the sheet: C14, C15, J1, L3

Commit message: speek rx schematic improvements
Parts:
- added Q1, Q2: SS8050-G, easyeda2kicad:SOT-23-3_L2.9-W1.5-P1.90-LS2.6-BR, symbol lcsc:SS8050-G_C3199946
- added R10, R11: 10k, easyeda2kicad:R0402, symbol lcsc:RC0402FR-0710KL
- R3: value RC0402FR-0710KL -> 10k
Connections:
- net CHIP_PU: now also Q1.3 (C); no longer J3.4 (Pin_4), U3.19 (RTS)
- net DTR: now also Q2.2 (E), R10.2; no longer BOOT1.2 (B), BOOT1.4 (D), C18.1, U1.23 (GPIO0)
- new net: Q2.1 (B), R11.1
- new net: Q1.1 (B), R10.1
- new net GPIO0: BOOT1.2 (B), BOOT1.4 (D), C18.1, Q2.3 (C), U1.23 (GPIO0)
- new net RTS: J3.4 (Pin_4), Q1.2 (E), R11.2, U3.19 (RTS)
Other:
- note added: "Antenna"
- note added: "Boot and EN buttons"
- note added: "DAC"
- note added: "ESP chip"
- note added: "Flash"
- note added: "Headphone amp"
- note added: "Output audio ports"
- note added: "Power / global"
- note added: "USB port"
- note added: "Uart converter"
- note removed: "No transistor circuit on purpose! It's just bloat, I have a good serial terminal"
- moved on the sheet: AE1, BOOT1, C1, C10, C11, C12, C13, C14, C15, C16, C17, C18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

Commit message: speek RX new board!!
Parts:
- removed C1, C13, C8: 1uF, lcsc:C0402, symbol lcsc:CL05A105KO5NNNC
- removed C10, C11: 15pf, lcsc:C0402, symbol lcsc:CL05C150JB5NNNC
- removed C12, C17, C2, C3, C5: 0.1uF, lcsc:C0402, symbol lcsc:CC0402KRX7R7BB104
- removed C14: GRM1555C1H2R7BA01D, easyeda2kicad:C0402, symbol lcsc:GRM1555C1H2R7BA01D
- removed C15: GRM1555C1H2R0BA01D, easyeda2kicad:C0402, symbol lcsc:GRM1555C1H2R0BA01D
- removed C4: 10uF, lcsc:C0402, symbol lcsc:CL05A106MP5NUNC_C15525
- removed C6: CC0402KRX7R9BB103, easyeda2kicad:C0402, symbol lcsc:CC0402KRX7R9BB103
- removed C7: CC0402KRX7R9BB332, easyeda2kicad:C0402, symbol lcsc:CC0402KRX7R9BB332
- removed C9: CC0402JRNPO9BN101, easyeda2kicad:C0402, symbol lcsc:CC0402JRNPO9BN101
- removed L1: LQG15HS2N0S02D, easyeda2kicad:L0402, symbol lcsc:LQG15HS2N0S02D
- removed L2: 15nH, lcsc:L0402, symbol lcsc:SDCL1005C15NJTDF
- removed L3: LQG15HS2N7S02D, easyeda2kicad:L0402, symbol lcsc:LQG15HS2N7S02D
- removed R1: RC-02K2002FT, easyeda2kicad:R0402, symbol lcsc:RC-02K2002FT
- removed R2: 499Ω, lcsc:R0402, symbol lcsc:FRC0402F4990TS
- removed R3: 10k, easyeda2kicad:R0402, symbol lcsc:RC0402FR-0710KL
- removed U1: ESP32-D0WD-V3, easyeda2kicad:QFN-48_L5.0-W5.0-P0.35-BL-EP3.7, symbol lcsc:ESP32-D0WD-V3
- removed U2: W25Q32JVSSIQ_C179173, easyeda2kicad:SOIC-8_L5.3-W5.3-P1.27-LS8.0-BL, symbol lcsc:W25Q32JVSSIQ_C179173
- removed X1: XL2EL89CPI-111YLC-40M, lcsc:CRYSTAL-SMD_4P-L3.2-W2.5-BL, symbol lcsc:XL2EL89CPI-111YLC-40M
- added C39: 0.1uF, lcsc:C0402, symbol lcsc:CC0402KRX7R7BB104
- added C40: 10uF, lcsc:C0402, symbol lcsc:CL05A106MP5NUNC_C15525
- added U19: ESP32-PICO-V3-02, easyeda2kicad:QFN-48_L7.0-W7.0-P0.50-BL-EP5.1, symbol lcsc:ESP32-PICO-V3-02
Connections:
- net BCK: now also U19.15 (IO26)
- net CHIP_PU: now also U19.9 (EN)
- net DIN: now also U19.39 (IO22)
- net GND: now also C39.1, C40.1, U19.49 (GND)
- net GPIO0: now also U19.23 (IO0)
- net GPIO25: now also U19.14 (IO25)
- net LNA_IN: now also JP1.1 (SIG), R9.2, U19.2 (LNA_IN)
- net PVDD: now also C39.2, C40.2, U19.1 (VDDA), U19.19 (VDD3P3_RTC), U19.3 (VDDA3P3), U19.37 (VDD3P3_CPU), U19.4 (VDDA3P3), U19.43 (VDDA), U19.46 (VDDA)
- net U0RXD: now also U19.40 (U0RXD/IO3)
- net U0TXD: now also U19.41 (U0TXD/IO1)
- no-connect marks 7 -> 19
Other:
- note removed: "Flash"

Commit message: aguihegwroiughawrg
Parts:
- removed D3, D4: PMEG060V100EPDZ, easyeda2kicad:SOT1289_L5.8-W4.4-LS6.5-RD, symbol lcsc:PMEG060V100EPDZ
- removed J1: Conn_01x02, Connector_JST:JST_VH_B2P-VH-B_1x02_P3.96mm_Vertical, symbol Connector_Generic:Conn_01x02
- C30, C31, C36, C37: value CL05A225KO5NQNC -> CL05A225MQ5NSNC; symbol lcsc:CL05A225KO5NQNC -> lcsc:CL05A225MQ5NSNC; LCSC Part C170151 -> C12530; MPN CL05A225KO5NQNC -> CL05A225MQ5NSNC
- C38: LCSC Part C1550 -> C309455; MPN 0402CG1R0C500NT -> CC0402BRNPO9BN1R0; Manufacturer Guangdong Fenghua(风华高科) -> YAGEO(国巨)
- D2: value PESD3V3L1BA,115 -> PESD3V3L1BA; symbol lcsc:PESD3V3L1BA,115 -> lcsc:PESD3V3L1BA; LCSC Part C51450 -> C2827682; MPN PESD3V3L1BA,115 -> PESD3V3L1BA; Manufacturer Nexperia(安世) -> TECH PUBLIC
- Q1, Q2: value SS8050-G -> SS8050; symbol lcsc:SS8050-G_C3199946 -> lcsc:SS8050_C2150; LCSC Part C3199946 -> C2150; MPN SS8050-G -> SS8050(RANGE:200-350); Manufacturer Comchip(典琦) -> JSCJ(江苏长电)
- R10, R11: symbol lcsc:RC0402FR-0710KL -> lcsc:0402WGF1002TCE; MPN RC0402FR-0710KL -> 0402WGF1002TCE; Manufacturer YAGEO(国巨) -> UNI-ROYAL(厚声)
- R5: value AR02DTD4752 -> 47k; symbol lcsc:AR02DTD4752 -> lcsc:0402WGF4702TCE; LCSC Part C319604 -> C25792; MPN AR02DTD4752 -> 0402WGF4702TCE; Manufacturer Viking(光颉) -> UNI-ROYAL(厚声)
- R6: value CRCW040222K1FKED -> 22k; symbol lcsc:CRCW040222K1FKED -> lcsc:0402WGF2202TCE; LCSC Part C844504 -> C25768; MPN CRCW040222K1FKED -> 0402WGF2202TCE; Manufacturer VISHAY(威世) -> UNI-ROYAL(厚声)
- R7: value RC0402FR-0710KL -> 10k; symbol lcsc:RC0402FR-0710KL -> lcsc:0402WGF1002TCE; MPN RC0402FR-0710KL -> 0402WGF1002TCE; Manufacturer YAGEO(国巨) -> UNI-ROYAL(厚声)
- R9: value RC0603JR-070RL -> 0R; symbol lcsc:RC0603JR-070RL -> lcsc:0603WAF0000T5E; LCSC Part C95177 -> C21189; MPN RC0603JR-070RL -> 0603WAF0000T5E; Manufacturer YAGEO(国巨) -> UNI-ROYAL(厚声)
- U4: value SPX1117M3-L-3-3/TR -> AMS1117-3.3; symbol lcsc:SPX1117M3-L-3-3_TR -> lcsc:AMS1117-3.3; LCSC Part C6862 -> C6186; MPN SPX1117M3-L-3-3/TR -> AMS1117-3.3; Manufacturer MaxLinear(迈凌) -> AMS(Advanced Monolithic Systems)
Connections:
- net __VIN is gone; now on net VBUS: J3.2 (Pin_2), U4.3 (input)
