File: speek-psu/PCB/speek_psu/speek_psu.kicad_pcb (KiCad board)
At the start: 2 copper layers, 80 x 60 mm, 21 parts, among them J1 Conn_01x02, J2 Conn_01x02, J3 Conn_01x02, J4 Conn_01x02, J5 Conn_01x02, J6 Conn_01x02, J7 Conn_01x02, J8 Conn_01x02, J9 Conn_01x02, U1 10k, U2 CH224K

Commit message: text
Other:
- board text added: "Speek PSU"
Changed lines of the file:
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@@
 				(font
 					(size 1.27 1.27)
+					(thickness 0.15)
 				)
 			)
@@
 				(font
 					(size 1.27 1.27)
+					(thickness 0.15)
 				)
 			)
@@
 				(font
 					(size 1.27 1.27)
+					(thickness 0.15)
 				)
 			)
@@
 				(font
 					(size 1.27 1.27)
+					(thickness 0.15)
 				)
 			)
@@
 				(font
 					(size 1.27 1.27)
+					(thickness 0.15)
 				)
 			)
@@
 				(font
 					(size 1.27 1.27)
+					(thickness 0.15)
 				)
 			)
@@
 				(font
 					(size 1.27 1.27)
+					(thickness 0.15)
 				)
 			)
@@
 				(font
 					(size 1.27 1.27)
+					(thickness 0.15)
 				)
 			)
@@
 		(layer "Edge.Cuts")
 	)
+	(gr_text "Speek PSU"
+		(at 121 78.25 0)
+		(layer "F.SilkS")
+		(effects
+			(font
+				(size 6 6)
+				(thickness 1)
+				(bold yes)
+			)
+			(justify left bottom)
+		)
+	)
 	(segment
 		(start 108.55 90.88)
@@
 	)
 	(segment
+		(start 108.55 90.08)
+		(end 109.92 90.08)
+		(width 0.55)
+		(layer "F.Cu")
+		(net "/VBUS")
+	)
+	(segment
+		(start 108.55 85.28)
+		(end 109.72 85.28)
+		(width 0.55)
+		(layer "F.Cu")
+		(net "/VBUS")
+	)
+	(segment
+		(start 118 93)
+		(end 118 91)
+		(width 0.2)
+		(layer "F.Cu")
+		(net "Net-(U2-VBUS)")
+	)
+	(segment
 		(start 121 111.5)
 		(end 121.2 111.7)
@@
 	)
 	(segment
-		(start 123 113)
-		(end 121 113)
+		(start 114.595 87.405)
+		(end 115.95 86.05)
 		(width 0.2)
 		(layer "F.Cu")
-		(net "Net-(LED1-A)")
+		(net "/D+")
 	)
 	(segment
-		(start 120 91)
-		(end 123 94)
+		(start 109.35 87.43)
+		(end 109.4 87.48)
 		(width 0.2)
 		(layer "F.Cu")
-		(net "/PG")
+		(net "/D+")
 	)
 	(segment
-		(start 123 94)
-		(end 123 110.9)
+		(start 109.375001 87.43)
+		(end 109.400001 87.405)
 		(width 0.2)
 		(layer "F.Cu")
-		(net "/PG")
+		(net "/D+")
 	)
 	(segment
-		(start 108.55 90.08)
-		(end 109.92 90.08)
-		(width 0.55)
+		(start 116.6 85.4)
+		(end 117 85)
+		(width 0.2)
 		(layer "F.Cu")
-		(net "/VBUS")
+		(net "/D+")
 	)
 	(segment
-		(start 108.55 85.28)
-		(end 109.72 85.28)
-		(width 0.55)
+		(start 108.55 87.43)
+		(end 109.375001 87.43)
+		(width 0.2)
 		(layer "F.Cu")
-		(net "/VBUS")
+		(net "/D+")
 	)
 	(segment
-		(start 120 93.14)
-		(end 119 92.14)
+		(start 109.400001 87.405)
+		(end 114.595 87.405)
 		(width 0.2)
 		(layer "F.Cu")
-		(net "Net-(U2-CFG1)")
+		(net "/D+")
 	)
 	(segment
-		(start 119 92.14)
-		(end 119 91)
+		(start 109.4 87.48)
+		(end 109.4 88.38)
 		(width 0.2)
 		(layer "F.Cu")
-		(net "Net-(U2-CFG1)")
+		(net "/D+")
 	)
 	(segment
-		(start 118 93)
-		(end 118 91)
+		(start 116.6 86.05)
+		(end 116.6 85.4)
 		(width 0.2)
 		(layer "F.Cu")
-		(net "Net-(U2-VBUS)")
+		(net "/D+")
+	)
+	(segment
+		(start 115.95 86.05)
+		(end 116.6 86.05)
+		(width 0.2)
+		(layer "F.Cu")
+		(net "/D+")
+	)
+	(segment
+		(start 109.35 88.43)
+		(end 108.55 88.43)
+		(width 0.2)
+		(layer "F.Cu")
+		(net "/D+")
+	)
+	(segment
+		(start 109.4 88.38)
+		(end 109.35 88.43)
+		(width 0.2)
+		(layer "F.Cu")
+		(net "/D+")
+	)
+	(segment
+		(start 108.55 87.43)
+		(end 109.35 87.43)
+		(width 0.2)
+		(layer "F.Cu")
+		(net "/D+")
 	)
 	(segment
@@
 	)
 	(segment
-		(start 114.595 87.405)
-		(end 115.95 86.05)
-		(width 0.2)
-		(layer "F.Cu")
-		(net "/D+")
-	)
-	(segment
-		(start 109.35 87.43)
-		(end 109.4 87.48)
-		(width 0.2)
-		(layer "F.Cu")
-		(net "/D+")
-	)
-	(segment
-		(start 109.375001 87.43)
-		(end 109.400001 87.405)
-		(width 0.2)
-		(layer "F.Cu")
-		(net "/D+")
-	)
-	(segment
-		(start 116.6 85.4)
-		(end 117 85)
-		(width 0.2)
-		(layer "F.Cu")
-		(net "/D+")
-	)
-	(segment
-		(start 108.55 87.43)
-		(end 109.375001 87.43)
-		(width 0.2)
-		(layer "F.Cu")
-		(net "/D+")
-	)
-	(segment
-		(start 109.400001 87.405)
-		(end 114.595 87.405)
-		(width 0.2)
-		(layer "F.Cu")
-		(net "/D+")
-	)
-	(segment
-		(start 109.4 87.48)
-		(end 109.4 88.38)
-		(width 0.2)
-		(layer "F.Cu")
-		(net "/D+")
-	)
-	(segment
-		(start 116.6 86.05)
-		(end 116.6 85.4)
+		(start 120 93.14)
+		(end 119 92.14)
 		(width 0.2)
 		(layer "F.Cu")
-		(net "/D+")
+		(net "Net-(U2-CFG1)")
 	)
 	(segment
-		(start 115.95 86.05)
-		(end 116.6 86.05)
+		(start 119 92.14)
+		(end 119 91)
 		(width 0.2)
 		(layer "F.Cu")
-		(net "/D+")
+		(net "Net-(U2-CFG1)")
 	)
 	(segment
-		(start 109.35 88.43)
-		(end 108.55 88.43)
+		(start 120 91)
+		(end 123 94)
 		(width 0.2)
 		(layer "F.Cu")
-		(net "/D+")
+		(net "/PG")
 	)
 	(segment
-		(start 109.4 88.38)
-		(end 109.35 88.43)
+		(start 123 94)
+		(end 123 110.9)
 		(width 0.2)
 		(layer "F.Cu")
-		(net "/D+")
+		(net "/PG")
 	)
 	(segment
-		(start 108.55 87.43)
-		(end 109.35 87.43)
+		(start 123 113)
+		(end 121 113)
 		(width 0.2)
 		(layer "F.Cu")
-		(net "/D+")
+		(net "Net-(LED1-A)")
 	)
 	(zone

Commit message: JST and antenna
Parts:
- added D1: PMEG060V100EPDZ, easyeda2kicad:SOT1289_L5.8-W4.4-LS6.5-RD, F.Cu at (116.5, 92.5)
- added D2: PMEG060V100EPDZ, easyeda2kicad:SOT1289_L5.8-W4.4-LS6.5-RD, F.Cu at (119.3, 64.5)
- added U3: 25PX4700MEFC16X25, easyeda2kicad:CAP-TH_BD16.0-P7.50-D1.2-FD, F.Cu at (154.8, 84.0)
- added U4: XT60, easyeda2kicad:CONN-TH_XT60, B.Cu at (107.0, 95.6)
- J1, J2, J3, J4, J5, J6, J7, J8: footprint Connector_JST:JST_EH_S2B-EH_1x02_P2.50mm_Horizontal -> Connector_JST:JST_VH_B2P-VH-B_1x02_P3.96mm_Vertical
- moved J7 53.1 mm to (179.2, 106.0), turned to 90 degrees
- moved J5 33.7 mm to (179.2, 96.5), turned to 90 degrees
- moved J1 25.1 mm to (157.5, 61.2), turned to 180 degrees
- moved J3 12.2 mm to (179.2, 77.5), turned to 90 degrees
- moved J4 11.7 mm to (179.2, 87.0), turned to 90 degrees
- moved J2 11.5 mm to (167.2, 61.2), turned to 180 degrees
- moved USB1 10.6 mm to (106.4, 77.1)
- moved C1 10.6 mm to (122.5, 74.4)
- moved R1 10.6 mm to (119.2, 70.4)
- moved R3 10.6 mm to (120.2, 83.0)
- moved U1 10.6 mm to (118.2, 83.4)
- moved U2 10.6 mm to (118.2, 77.4)
- moved J6 7.84 mm to (148.0, 61.2), turned to 180 degrees
- moved J8 6.78 mm to (138.5, 61.2), turned to 180 degrees
Connections:
- J1 pad 2: /VBUS -> /_VOUT
- J2 pad 2: /VBUS -> /_VOUT
- J3 pad 2: /VBUS -> /_VOUT
- J4 pad 2: /VBUS -> /_VOUT
- J5 pad 2: /VBUS -> /_VOUT
- J6 pad 2: /VBUS -> /_VOUT
- J7 pad 2: /VBUS -> /_VOUT
- J8 pad 2: /VBUS -> /_VOUT
- J9 pad 2: /VBUS -> /_VOUT
Routing:
- net /VBUS: track 2.54 -> 60.5 mm
- net /PG: track 21.1 -> 33.7 mm
- net /_VOUT: track 0.00 -> 11.6 mm
- net /VDD: track 41.4 -> 49.3 mm
- net Net-(U4-+): track 0.00 -> 6.56 mm
- added copper zone on F.Cu, net /_VOUT
- removed copper zone on F.Cu, net /VBUS

Commit message: connectors
Parts:
- added U5: 50PX4700MEFC18X40, easyeda2kicad:CAP-TH_BD18.0-P7.50-D0.8-FD, F.Cu at (155.0, 83.2)
- added U6: ~, easyeda2kicad:CONN-TH_DB301V-3.5-2P-GN, F.Cu at (151.7, 111.8)
- added U7: ~, easyeda2kicad:CONN-TH_DB301V-3.5-2P-GN, F.Cu at (160.2, 111.8)
- added U8: ~, easyeda2kicad:CONN-TH_DB301V-3.5-2P-GN, F.Cu at (169.0, 111.8)
- U3: value 25PX4700MEFC16X25 -> ~; footprint easyeda2kicad:CAP-TH_BD16.0-P7.50-D1.2-FD -> easyeda2kicad:CONN-TH_DB301V-3.5-2P-GN
- U4: moved to F.Cu
- moved U3 30.2 mm to (142.8, 111.8), turned to 0 degrees
Connections:
- U3 pad 1: /_VOUT -> GND
- U3 pad 2: GND -> /_VOUT

Commit message: Speek PSU no longer requires PCBA !!
Parts:
- removed C1: 1uf, easyeda2kicad:C0603
- removed D1, D2: PMEG060V100EPDZ, easyeda2kicad:SOT1289_L5.8-W4.4-LS6.5-RD
- removed LED1: 0805G, easyeda2kicad:LED0805-R-RD
- removed R1: 1k, easyeda2kicad:R2010
- removed R2: 270Ω, easyeda2kicad:R0603
- removed R3: 200k, easyeda2kicad:R0402
- removed U1: 10k, easyeda2kicad:R0805
- removed U2: CH224K, easyeda2kicad:ESSOP-10_L4.9-W3.9-P1.0-LS6.0-TL-EP
- removed USB1: TYPE-C 16PIN 2MD, easyeda2kicad:USB-C-SMD_TYPE-C-16PIN-2MD-073
- added D3: 5KP100A, easyeda2kicad:DIO-TH_BD8.8-L8.8-P12.8-D1.6-RD, F.Cu at (129.4, 74.2)
- added J10: Conn_02x05_Counter_Clockwise, Connector_PinHeader_2.54mm:PinHeader_2x05_P2.54mm_Horizontal, F.Cu at (105.1, 71.9)
- moved J9 8.66 mm to (122.4, 113.2)
Connections:
- U4 pad 2: Net-(U4-+) -> /_VOUT
Routing:
- net /VDD: track 49.3 -> 0.00 mm
- net /PG: track 33.7 -> 0.00 mm
- net /VBUS: track 60.5 -> 29.1 mm
- net /CC1: track 13.7 -> 0.00 mm, vias 2 -> 0
- net /D+: track 12.5 -> 0.00 mm
- net /D-: track 11.1 -> 0.00 mm
- net /CC2: track 8.10 -> 0.00 mm
- net Net-(U4-+): track 6.56 -> 0.00 mm
- net /_VOUT: track 11.6 -> 18.1 mm
- net GND: track 4.70 -> 0.00 mm, vias 3 -> 0
- net Net-(U2-CFG1): track 2.55 -> 0.00 mm
- net Net-(U2-VBUS): track 2.00 -> 0.00 mm
- net Net-(LED1-A): track 2.00 -> 0.00 mm
Other:
- board text added: "+"
- board text added: "-"
