File: speek-amp/PCB/speek_amp/speek_amp.kicad_pcb (KiCad board)
At the start: 2 copper layers, 120 x 80 mm, 104 parts, among them U1 TPA3116D2DAD_C2865736, U10 TPA3116D2DAD_C2865736, U11 R_Tweeter, U12 R_Woofer, U13 10uH, U14 10uH, U15 L_Tweeter, U16 L_Woofer, U17 L_Sub, U18 J1, U2 10uH, U3 10uH, U4 XT60, U5 10uH, U6 10uH, U7 PDMTAT068125-151MLU, U8 PDMTAT068125-151MLU, U9 50PX4700MEFC18X40

Commit message: amp
Parts:
- removed D1, D2: PMEG060V100EPDZ, easyeda2kicad:SOT1289_L5.8-W4.4-LS6.5-RD
Connections:
- U18 pad 2: Net-(D2-A-Pad1) -> /VCC
- U4 pad 2: Net-(U4-+) -> /VCC
Routing:
- net /VCC: track 233.2 -> 252.9 mm
- net Net-(D2-A-Pad1): track 9.68 -> 0.00 mm
- net Net-(U4-+): track 6.59 -> 0.00 mm
- net /AMP_NR: track 44.7 -> 44.0 mm

Commit message: wowoowww
Parts:
- turned U1 to 90 degrees
- turned U10 to 90 degrees

Commit message: redoc
Parts:
- turned U1 to -90 degrees
- turned U10 to -90 degrees
